File: VoltageSources.kicad_sch (KiCad schematic)
At the start: 19 parts, among them J10 Conn_01x01_Socket, J11 Conn_01x02_Socket, J12 Conn_01x03_Socket, J13 Lever Terminal, J7 USB_C_Receptacle_PowerOnly_6P, J8 Conn_01x01_Socket, J9 Conn_01x01_Socket, SW14 SW_SPST, U6 MEE3S0505SC

Commit message: preliminary layout of op amp blocks complete
Parts:
- added U7: TPS61175PWP, PWP14_2P31X2P46, symbol TPS61175:TPS61175PWP
Changed lines of the file:
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@@
+	)
+	(symbol
+		(lib_id "TPS61175:TPS61175PWP")
+		(at 170.18 55.88 0)
+		(unit 1)
+		(body_style 1)
+		(exclude_from_sim no)
+		(in_bom yes)
+		(on_board yes)
+		(in_pos_files yes)
+		(dnp no)
+		(fields_autoplaced yes)
+		(property "Reference" "U7"
+			(at 200.66 45.72 0)
+			(show_name no)
+			(do_not_autoplace no)
+			(effects
+				(font
+					(size 1.524 1.524)
+				)
+			)
+		)
+		(property "Value" "TPS61175PWP"
+			(at 200.66 48.26 0)
+			(show_name no)
+			(do_not_autoplace no)
+			(effects
+				(font
+					(size 1.524 1.524)
+				)
+			)
+		)
+		(property "Footprint" "PWP14_2P31X2P46"
+			(at 170.18 55.88 0)
+			(hide yes)
+			(show_name no)
+			(do_not_autoplace no)
+			(effects
+				(font
+					(size 1.27 1.27)
+					(italic yes)
+				)
+			)
+		)
+		(property "Datasheet" "https://www.ti.com/lit/gpn/tps61175"
+			(at 170.18 55.88 0)
+			(hide yes)
+			(show_name no)
+			(do_not_autoplace no)
+			(effects
+				(font
+					(size 1.27 1.27)
+					(italic yes)
+				)
+			)
+		)
+		(property "Description" ""
+			(at 170.18 55.88 0)
+			(hide yes)
+			(show_name no)
+			(do_not_autoplace no)
+			(effects
+				(font
+					(size 1.27 1.27)
+				)
+			)
+		)
+		(pin "8"
+		)
+		(pin "5"
+		)
+		(pin "14"
+		)
+		(pin "9"
+		)
+		(pin "3"
+		)
+		(pin "15"
+		)
+		(pin "13"
+		)
+		(pin "11"
+		)
+		(pin "12"
+		)
+		(pin "10"
+		)
+		(pin "7"
+		)
+		(pin "6"
+		)
+		(pin "1"
+		)
+		(pin "2"
+		)
+		(pin "4"
+		)
+		(instances
+			(project "universalOpAmpV0"
+				(path "/0c9d5097-e341-4aa8-a29f-4bc5e653f52f/604e846a-aad5-4cbc-a3c9-ff0e9d7c3047"
+					(reference "U7")
+					(unit 1)
+				)
+			)
+		)
 	)
 	(symbol
