File: universalOpAmpV0.kicad_pcb (KiCad board)
At the start: 6 copper layers, 142.8 x 74.7 mm, 127 parts, among them J1 BNC I1, J2 BNC I1, J3 BNC I1, J4 BNC I1, J5 BNC I1, J6 BNC I1, SW1 218-8LPSTR, SW15 218-4LPSTR, SW16 SW_DPDT, SW17 SW_DPDT, SW18 CS-4-14, SW19 SW_SP3T, SW20 218-8LPSTR, SW21 218-4LPSTR, SW22 SW_DPDT, SW23 SW_DPDT, SW24 CS-4-14, SW25 SW_SP3T, SW26 218-8LPSTR, SW27 218-4LPSTR, SW28 SW_DPDT, SW29 SW_DPDT, SW3 218-4LPSTR, SW30 CS-4-14, SW31 SW_SP3T, SW32 218-8LPSTR, SW33 218-4LPSTR, SW34 SW_DPDT, SW35 SW_DPDT, SW36 CS-4-14, SW37 SW_SP3T, SW38 218-8LPSTR, SW39 218-4LPSTR, SW4 SW_DPDT, SW40 SW_DPDT, SW41 SW_DPDT, SW42 CS-4-14, SW43 SW_SP3T, SW45 218-8LPSTR, SW47 218-8LPSTR, SW49 218-8LPSTR, SW5 SW_DPDT, SW6 CS-4-14, SW7 SW_SP3T, SW8 218-8LPSTR, U1 OPA992DBV, U10 OPA992DBV, U13 OPA992DBV, U14 OPA992DBV, U2 BUF634A, U3 OPA992DBV, U4 OPA992DBV, U5 BUF634A, U8 OPA992DBV, U9 OPA992DBV

Commit message: input stage schematic done, layout WIP
Parts:
- added C76: 100n, uniOpAmpLib:PP_CAP, F.Cu at (119.1, 43.9)
- added C78: 100n, uniOpAmpLib:PP_CAP, F.Cu at (71.0, 92.6)
- added C79: 100n, uniOpAmpLib:PP_CAP, F.Cu at (110.0, 119.6)
- added C80: C, uniOpAmpLib:C_0805_Metric2012_HandSolder, F.Cu at (101.4, 42.6)
- added C81: C, uniOpAmpLib:C_0805_Metric2012_HandSolder, F.Cu at (101.4, 45.6)
- added C82: C, uniOpAmpLib:C_0805_Metric2012_HandSolder, F.Cu at (101.4, 48.6)
- added C83: C, uniOpAmpLib:C_0805_Metric2012_HandSolder, F.Cu at (101.4, 51.6)
- added C84: C, uniOpAmpLib:C_0805_Metric2012_HandSolder, F.Cu at (101.4, 54.6)
- added C85: C, uniOpAmpLib:C_0805_Metric2012_HandSolder, F.Cu at (101.4, 57.7)
- added C86: C, uniOpAmpLib:C_0805_Metric2012_HandSolder, F.Cu at (53.3, 91.4)
- added C87: C, uniOpAmpLib:C_0805_Metric2012_HandSolder, F.Cu at (53.3, 94.4)
- added C88: C, uniOpAmpLib:C_0805_Metric2012_HandSolder, F.Cu at (53.3, 97.4)
- added C89: C, uniOpAmpLib:C_0805_Metric2012_HandSolder, F.Cu at (53.3, 100.4)
- added C90: C, uniOpAmpLib:C_0805_Metric2012_HandSolder, F.Cu at (53.3, 103.4)
- added C91: C, uniOpAmpLib:C_0805_Metric2012_HandSolder, F.Cu at (53.3, 106.4)
- added C92: C, uniOpAmpLib:C_0805_Metric2012_HandSolder, F.Cu at (111.9, 109.6)
- added C93: C, uniOpAmpLib:C_0805_Metric2012_HandSolder, B.Cu at (87.4, 112.5)
- added C94: C, uniOpAmpLib:C_0805_Metric2012_HandSolder, B.Cu at (92.2, 112.8)
- added C95: C, uniOpAmpLib:C_0805_Metric2012_HandSolder, B.Cu at (91.2, 116.1)
- added C96: C, uniOpAmpLib:C_0805_Metric2012_HandSolder, B.Cu at (87.4, 115.1)
- added C97: C, uniOpAmpLib:C_0805_Metric2012_HandSolder, F.Cu at (115.0, 114.1)
- added R10: 1M, Resistor_SMD:R_0805_2012Metric_Pad1.20x1.40mm_HandSolder, F.Cu at (58.0, 91.3)
- added R11: 1M, Resistor_SMD:R_0805_2012Metric_Pad1.20x1.40mm_HandSolder, F.Cu at (98.6, 118.1)
- added R12: R, Resistor_SMD:R_0805_2012Metric_Pad1.20x1.40mm_HandSolder, F.Cu at (106.1, 45.5)
- added R13: R, Resistor_SMD:R_0805_2012Metric_Pad1.20x1.40mm_HandSolder, F.Cu at (58.0, 94.3)
- added R14: R, Resistor_SMD:R_0805_2012Metric_Pad1.20x1.40mm_HandSolder, F.Cu at (109.0, 113.5)
- added R15: R, Resistor_SMD:R_0805_2012Metric_Pad1.20x1.40mm_HandSolder, F.Cu at (106.1, 48.5)
- added R16: R, Resistor_SMD:R_0805_2012Metric_Pad1.20x1.40mm_HandSolder, F.Cu at (58.0, 97.2)
- added R17: R, Resistor_SMD:R_0805_2012Metric_Pad1.20x1.40mm_HandSolder, F.Cu at (131.6, 106.7)
- added R18: R, Resistor_SMD:R_0805_2012Metric_Pad1.20x1.40mm_HandSolder, F.Cu at (106.1, 51.4)
- added R19: R, Resistor_SMD:R_0805_2012Metric_Pad1.20x1.40mm_HandSolder, F.Cu at (58.0, 100.2)
- added R20: R, Resistor_SMD:R_0805_2012Metric_Pad1.20x1.40mm_HandSolder, F.Cu at (131.6, 108.7)
- added R21: R, Resistor_SMD:R_0805_2012Metric_Pad1.20x1.40mm_HandSolder, F.Cu at (106.1, 54.4)
- added R22: R, Resistor_SMD:R_0805_2012Metric_Pad1.20x1.40mm_HandSolder, F.Cu at (58.0, 103.1)
- added R23: R, Resistor_SMD:R_0805_2012Metric_Pad1.20x1.40mm_HandSolder, F.Cu at (131.6, 110.7)
- added R24: 50R, Resistor_SMD:R_2512_6332Metric_Pad1.40x3.35mm_HandSolder, F.Cu at (119.1, 52.4)
- added R25: 50R, Resistor_SMD:R_2512_6332Metric_Pad1.40x3.35mm_HandSolder, F.Cu at (71.0, 101.1)
- added R26: 50R, Resistor_SMD:R_2512_6332Metric_Pad1.40x3.35mm_HandSolder, B.Cu at (100.6, 115.3)
- added R27: 0R, Resistor_SMD:R_0805_2012Metric_Pad1.20x1.40mm_HandSolder, F.Cu at (106.1, 57.3)
- added R28: 0R, Resistor_SMD:R_0805_2012Metric_Pad1.20x1.40mm_HandSolder, F.Cu at (58.0, 106.1)
- added R29: 0R, Resistor_SMD:R_0805_2012Metric_Pad1.20x1.40mm_HandSolder, F.Cu at (119.6, 122.2)
- added R7: 1M, Resistor_SMD:R_0805_2012Metric_Pad1.20x1.40mm_HandSolder, F.Cu at (106.1, 42.6)
- added SW11: SW_Rotary_1x7, uniOpAmpLib:SS-10-16, F.Cu at (232.7, 99.0)
- added SW11: SW_Rotary_1x7, uniOpAmpLib:SS-10-16, F.Cu at (232.7, 87.0)
- added SW11: SW_Rotary_1x7, uniOpAmpLib:SS-10-16, F.Cu at (232.7, 111.0)
- added SW44: SW_DIP_x02, uniOpAmpLib:218-2LPSTR, F.Cu at (51.0, 118.1)
- added SW46: SW_DIP_x02, uniOpAmpLib:218-2LPSTR, F.Cu at (43.9, 118.1)
- added SW48: SW_DIP_x02, uniOpAmpLib:218-2LPSTR, F.Cu at (115.1, 121.4)
- added SW50: SW_DPDT_x2, uniOpAmpLib:CAS-DxxB, F.Cu at (111.5, 53.7)
- added SW51: SW_DPDT_x2, uniOpAmpLib:CAS-DxxB, F.Cu at (63.4, 102.4)
- added SW52: SW_DPDT_x2, uniOpAmpLib:CAS-DxxB, F.Cu at (103.9, 116.6)
- added SW53: CS-4-14, uniOpAmpLib:CS-4-14NB, F.Cu at (111.7, 45.5)
- added SW54: CS-4-14, uniOpAmpLib:CS-4-14NB, F.Cu at (63.6, 94.3)
- added SW55: CS-4-14, uniOpAmpLib:CS-4-14NB, F.Cu at (125.7, 108.7)
- added U15: OPA992DBV, uniOpAmpLib:SOT-23-5_HandSoldering, F.Cu at (117.4, 57.3)
- added U16: OPA992DBV, uniOpAmpLib:SOT-23-5_HandSoldering, F.Cu at (69.3, 106.0)
- added U17: OPA992DBV, uniOpAmpLib:SOT-23-5_HandSoldering, F.Cu at (111.9, 113.1)
- moved U5 36.3 mm to (242.1, 83.8)
- moved J4 15.2 mm to (248.9, 74.9)
- moved J5 15.2 mm to (248.9, 99.9)
- moved J6 15.2 mm to (248.9, 124.9)
- moved C9 11.7 mm to (138.7, 87.9)
- moved C1 11.7 mm to (153.7, 89.4)
- moved C2 11.7 mm to (157.8, 87.9)
- moved C3 11.7 mm to (153.7, 87.4)
- moved C32 11.7 mm to (153.8, 105.6)
- moved C33 11.7 mm to (157.9, 104.1)
- moved C34 11.7 mm to (153.8, 103.6)
- moved C35 11.7 mm to (157.9, 104.1)
- moved C36 11.7 mm to (153.8, 105.6)
- moved C37 11.7 mm to (159.9, 104.1)
- moved C38 11.7 mm to (149.8, 104.1)
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Connections:
- SW1 pad 1: /InputStage1/I -> Net-(SW50A-B)
- SW1 pad 2: /InputStage1/I -> Net-(SW50A-B)
- SW1 pad 3: /InputStage1/I -> Net-(SW50A-B)
- SW1 pad 4: /InputStage1/I -> Net-(SW50A-B)
- SW1 pad 5: /InputStage1/I -> Net-(SW50A-B)
- SW1 pad 6: /InputStage1/I -> Net-(SW50A-B)
- SW1 pad 7: /InputStage1/I -> Net-(SW50A-B)
- SW1 pad 8: /InputStage1/I -> Net-(SW50A-B)
- SW47 pad 1: /InputStage2/I -> Net-(SW51A-B)
- SW47 pad 2: /InputStage2/I -> Net-(SW51A-B)
- SW47 pad 3: /InputStage2/I -> Net-(SW51A-B)
- SW47 pad 4: /InputStage2/I -> Net-(SW51A-B)
- SW47 pad 5: /InputStage2/I -> Net-(SW51A-B)
- SW47 pad 6: /InputStage2/I -> Net-(SW51A-B)
- SW47 pad 7: /InputStage2/I -> Net-(SW51A-B)
- SW47 pad 8: /InputStage2/I -> Net-(SW51A-B)
- SW49 pad 1: /InputStage3/I -> Net-(SW52A-B)
- SW49 pad 2: /InputStage3/I -> Net-(SW52A-B)
- SW49 pad 3: /InputStage3/I -> Net-(SW52A-B)
- SW49 pad 4: /InputStage3/I -> Net-(SW52A-B)
- SW49 pad 5: /InputStage3/I -> Net-(SW52A-B)
- SW49 pad 6: /InputStage3/I -> Net-(SW52A-B)
- SW49 pad 7: /InputStage3/I -> Net-(SW52A-B)
- SW49 pad 8: /InputStage3/I -> Net-(SW52A-B)
Routing:
- net /InputStage3/I: track 13.5 -> 0.00 mm
- net /InputStage1/I: track 13.5 -> 0.00 mm
- net /InputStage2/I: track 12.5 -> 0.00 mm
- net Net-(RV5-Pad1): track 26.6 -> 27.9 mm, vias 0 -> 1
- added copper zone on In3.Cu, net GND
- removed copper zone on In1.Cu, net GND
Other:
- board size 142.8 x 74.7 mm -> 151.7 x 74.7 mm
